File: PCB/MotorHall.kicad_sch (KiCad schematic)
At the start: 18 parts, among them U4 DRV8311S, U5 DRV5055A1xDBZxQ1

Commit message: Made various changes for increased readability
Parts:
- D66, R104, U6: now not fitted
Other:
- note added: "H1 and H2 are to be used if DC motor is used. Do do this, DNP R101 and R102 and populate FET U6 and R104"
- note added: "PWM Motor Control"
- note added: "SPI Motor Config."
- note removed: "H2 and H3 are to be used if DC motor is used. Do do this, DNP R102 and R103 and populate FET U6"
- company: (none) -> BYU IEEE Student Branch
- title: (none) -> Volumetric Display
- moved on the sheet: R65

Commit message: Generated release package X0
Parts:
- added FID1, FID2, FID3, FID4: Fiducial, Fiducial:Fiducial_0.5mm_Mask1mm, symbol Mechanical:Fiducial
- U6: value ~ -> (none)
