File: PCB/Programming.kicad_sch (KiCad schematic)
At the start: 13 parts, among them J1 USB_C_Receptacle_USB2.0_16P, U1 FT260S-R

Commit message: Made various changes for increased readability
Other:
- note added: "UART PROG. Interface"
- company: (none) -> BYU IEEE Student Branch
- title: (none) -> Volumetric Display
Changed lines of the file:
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@@
 	(generator_version "9.0")
 	(paper "A4")
+	(title_block
+		(title "Volumetric Display")
+		(rev "X0")
+		(company "BYU IEEE Student Branch")
+		(comment 1 "Design: Ryan H.")
+		(comment 2 "Drawn: Ryan H.")
+		(comment 3 "Reviewed: Nathan F.")
+	)
+	(text "UART PROG. Interface"
+		(exclude_from_sim no)
+		(at 184.658 98.806 0)
+		(effects
+			(font
+				(size 1.27 1.27)
+			)
+		)
+	)
 	(junction
 		(at 76.2 45.72)
@@
 	)
 	(junction
+		(at 148.59 82.55)
+		(diameter 0)
+		(color 0 0 0 0)
+	)
+	(junction
 		(at 74.93 77.47)
 		(diameter 0)
@@
 	)
 	(junction
-		(at 152.4 82.55)
-		(diameter 0)
-		(color 0 0 0 0)
-	)
-	(junction
 		(at 76.2 59.69)
 		(diameter 0)
@@
 	(wire
 		(pts
-			(xy 151.13 82.55) (xy 152.4 82.55)
+			(xy 147.32 82.55) (xy 148.59 82.55)
 		)
 		(stroke
@@
 	(wire
 		(pts
-			(xy 158.75 80.01) (xy 152.4 80.01)
+			(xy 158.75 80.01) (xy 148.59 80.01)
 		)
 		(stroke
@@
 	(wire
 		(pts
+			(xy 148.59 82.55) (xy 153.67 82.55)
+		)
+		(stroke
+			(width 0)
+			(type default)
+		)
+	)
+	(wire
+		(pts
 			(xy 199.39 69.85) (xy 201.93 69.85)
 		)
@@
 	(wire
 		(pts
-			(xy 152.4 80.01) (xy 152.4 82.55)
+			(xy 148.59 80.01) (xy 148.59 82.55)
 		)
 		(stroke
@@
 		(pts
 			(xy 199.39 90.17) (xy 201.93 90.17)
-		)
-		(stroke
-			(width 0)
-			(type default)
-		)
-	)
-	(wire
-		(pts
-			(xy 152.4 82.55) (xy 153.67 82.55)
 		)
 		(stroke
@@
 		(on_board yes)
 		(dnp no)
-		(fields_autoplaced yes)
 		(property "Reference" "#PWR014"
 			(at 149.86 62.23 0)
@@
 		)
 		(property "Value" "GND"
-			(at 152.4 62.2299 90)
+			(at 153.67 62.23 90)
 			(effects
 				(font
@@
 		(on_board yes)
 		(dnp no)
-		(fields_autoplaced yes)
 		(property "Reference" "#PWR07"
 			(at 53.34 109.22 0)
@@
 		)
 		(property "Value" "GND"
-			(at 53.34 107.95 0)
+			(at 53.34 106.426 0)
 			(effects
 				(font
@@
 		(on_board yes)
 		(dnp no)
-		(fields_autoplaced yes)
 		(property "Reference" "R73"
-			(at 157.48 76.2 90)
+			(at 153.162 81.534 90)
 			(effects
 				(font
@@
 		)
 		(property "Value" "0"
-			(at 157.48 78.74 90)
+			(at 160.274 81.534 90)
 			(effects
 				(font
@@
 		(on_board yes)
 		(dnp no)
-		(fields_autoplaced yes)
 		(property "Reference" "R98"
-			(at 78.74 36.8299 0)
+			(at 77.216 37.084 0)
 			(effects
 				(font
@@
 		)
 		(property "Value" "50K"
-			(at 78.74 39.3699 0)
+			(at 77.216 38.862 0)
 			(effects
 				(font
@@
 		(on_board yes)
 		(dnp no)
-		(fields_autoplaced yes)
 		(property "Reference" "R71"
-			(at 162.56 55.88 90)
+			(at 158.496 61.214 90)
 			(effects
 				(font
@@
 		)
 		(property "Value" "0"
-			(at 162.56 58.42 90)
+			(at 165.354 61.214 90)
 			(effects
 				(font
@@
 		(on_board yes)
 		(dnp no)
-		(fields_autoplaced yes)
 		(property "Reference" "R66"
-			(at 88.9 69.8499 0)
+			(at 87.376 70.104 0)
 			(effects
 				(font
@@
 		)
 		(property "Value" "5.1K"
-			(at 88.9 72.3899 0)
+			(at 87.376 71.882 0)
 			(effects
 				(font
@@
 		(on_board yes)
 		(dnp no)
-		(fields_autoplaced yes)
 		(property "Reference" "U1"
-			(at 184.15 55.88 0)
+			(at 184.15 57.658 0)
 			(effects
 				(font
@@
 		)
 		(property "Value" "FT260S-R"
-			(at 184.15 58.42 0)
+			(at 184.15 59.69 0)
 			(effects
 				(font
@@
 		(on_board yes)
 		(dnp no)
-		(fields_autoplaced yes)
 		(property "Reference" "J1"
-			(at 57.15 52.07 0)
+			(at 57.15 54.102 0)
 			(effects
 				(font
@@
 		)
 		(property "Value" "USB_C_Receptacle_USB2.0_16P"
-			(at 57.15 54.61 0)
+			(at 57.15 55.88 0)
 			(effects
 				(font
@@
 		(on_board yes)
 		(dnp no)
-		(fields_autoplaced yes)
 		(property "Reference" "R97"
-			(at 78.74 53.3399 0)
+			(at 77.216 53.594 0)
 			(effects
 				(font
@@
 		)
 		(property "Value" "50K"
-			(at 78.74 55.8799 0)
+			(at 77.216 55.372 0)
 			(effects
 				(font
@@
 		(on_board yes)
 		(dnp no)
-		(fields_autoplaced yes)
 		(property "Reference" "R67"
-			(at 97.79 67.3099 0)
+			(at 96.266 67.564 0)
 			(effects
 				(font
@@
 		)
 		(property "Value" "5.1K"
-			(at 97.79 69.8499 0)
+			(at 96.266 69.342 0)
 			(effects
 				(font
@@
 		(on_board yes)
 		(dnp no)
-		(fields_autoplaced yes)
 		(property "Reference" "R69"
-			(at 142.24 68.58 90)
+			(at 138.176 73.914 90)
 			(effects
 				(font
@@
 		)
 		(property "Value" "0"
-			(at 142.24 71.12 90)
+			(at 145.034 73.914 90)
 			(effects
 				(font
@@
 		(on_board yes)
 		(dnp no)
-		(fields_autoplaced yes)
 		(property "Reference" "R68"
-			(at 149.86 66.04 90)
+			(at 145.542 71.374 90)
 			(effects
 				(font
@@
 		)
 		(property "Value" "0"
-			(at 149.86 68.58 90)
+			(at 152.654 71.374 90)
 			(effects
 				(font
@@
 		(on_board yes)
 		(dnp no)
-		(fields_autoplaced yes)
 		(property "Reference" "D65"
-			(at 90.4875 53.34 0)
+			(at 90.17 57.404 0)
 			(effects
 				(font
@@
 		)
 		(property "Value" "MBR0560"
-			(at 90.4875 55.88 0)
+			(at 90.17 62.23 0)
 			(effects
 				(font
@@
 		(on_board yes)
 		(dnp no)
-		(fields_autoplaced yes)
 		(property "Reference" "R70"
-			(at 134.62 71.12 90)
+			(at 130.556 76.454 90)
 			(effects
 				(font
@@
 		)
 		(property "Value" "0"
-			(at 134.62 73.66 90)
+			(at 137.414 76.454 90)
 			(effects
 				(font
@@
 		(on_board yes)
 		(dnp no)
-		(fields_autoplaced yes)
 		(property "Reference" "#PWR08"
 			(at 95.25 83.82 0)
@@
 		)
 		(property "Value" "GND"
-			(at 95.25 82.55 0)
+			(at 95.25 81.026 0)
 			(effects
 				(font
@@
 		(on_board yes)
 		(dnp no)
-		(fields_autoplaced yes)
 		(property "Reference" "R72"
-			(at 162.56 73.66 90)
+			(at 158.242 78.994 90)
 			(effects
 				(font
@@
 		)
 		(property "Value" "0"
-			(at 162.56 76.2 90)
+			(at 165.354 78.994 90)
 			(effects
 				(font
@@
 		(on_board yes)
 		(dnp no)
-		(fields_autoplaced yes)
 		(property "Reference" "#PWR037"
 			(at 64.77 34.29 0)
@@
 		)
 		(property "Value" "GND"
-			(at 67.31 34.2899 90)
+			(at 68.326 34.29 90)
 			(effects
 				(font
@@
 	(symbol
 		(lib_id "power:GND")
-		(at 151.13 82.55 270)
+		(at 147.32 82.55 270)
 		(unit 1)
 		(exclude_from_sim no)
@@
 		(on_board yes)
 		(dnp no)
-		(fields_autoplaced yes)
 		(property "Reference" "#PWR017"
-			(at 144.78 82.55 0)
+			(at 140.97 82.55 0)
 			(effects
 				(font
@@
 		)
 		(property "Value" "GND"
-			(at 147.32 82.5499 90)
+			(at 144.78 82.55 90)
 			(effects
 				(font
@@
 		)
 		(property "Footprint" ""
-			(at 151.13 82.55 0)
+			(at 147.32 82.55 0)
 			(effects
 				(font
@@
 		)
 		(property "Datasheet" ""
-			(at 151.13 82.55 0)
+			(at 147.32 82.55 0)
 			(effects
 				(font
@@
 		)
 		(property "Description" "Power symbol creates a global label with name \"GND\" , ground"
-			(at 151.13 82.55 0)
-			(effects
-				(font
+			(at 147.32 82.55 0)
+			(effects
+				(font
