File: PCB/STM.kicad_sch (KiCad schematic)
At the start: 38 parts, among them U2 NCP718xSN330, U3 STM32G071R8T6

Commit message: Made various changes for increased readability
Other:
- note added: "Alt Prog."
- note added: "Motor & Speed Control"
- company: (none) -> BYU IEEE Student Branch
- title: (none) -> Volumetric Display

Commit message: Generated release package X0
Parts:
- TP1, TP2, TP3, TP4, TP5: now left out of the parts list
