File: PCB/VolumetricDisplay.kicad_sch (KiCad schematic)
At the start: 0 parts

Commit message: Made various changes for increased readability
Other:
- company: (none) -> BYU IEEE Student Branch
- title: (none) -> Volumetric Display
Changed lines of the file:
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@@
 	(generator_version "9.0")
 	(paper "A4")
-	(text_box "10 mA per LED:\n3V3 drive, 2V drop\n1.3V / 10 mA = 130 Ohms"
-		(exclude_from_sim no)
-		(at 15.24 183.515 0)
-		(size 30.48 8.255)
-		(margins 0.9525 0.9525 0.9525 0.9525)
-		(stroke
-			(width 0)
-			(type solid)
-		)
-		(fill
-			(type none)
-		)
-		(effects
-			(font
-				(size 1.27 1.27)
-			)
-			(justify left top)
-		)
+	(title_block
+		(title "Volumetric Display")
+		(date "2026-08-11")
+		(rev "X0")
+		(company "BYU IEEE Student Branch")
+		(comment 1 "Design: Ryan H.")
+		(comment 2 "Drawn: Ryan H.")
+		(comment 3 "Reviewed: Nathan F.")
 	)
 	(sheet
-		(at 120.015 28.575)
-		(size 20.32 14.605)
+		(at 151.13 69.85)
+		(size 27.94 20.32)
 		(exclude_from_sim no)
 		(in_bom yes)
@@
 		)
 		(property "Sheetname" "Programming"
-			(at 120.015 27.8634 0)
+			(at 151.13 69.1384 0)
 			(effects
 				(font
@@
 		)
 		(property "Sheetfile" "Programming.kicad_sch"
-			(at 120.015 43.7646 0)
+			(at 151.13 90.7546 0)
 			(effects
 				(font
@@
 	)
 	(sheet
-		(at 114.935 74.295)
-		(size 23.495 19.685)
+		(at 120.65 95.25)
+		(size 27.94 20.32)
 		(exclude_from_sim no)
 		(in_bom yes)
@@
 		)
 		(property "Sheetname" "STM"
-			(at 114.935 73.5834 0)
+			(at 120.65 94.5384 0)
 			(effects
 				(font
@@
 		)
 		(property "Sheetfile" "STM.kicad_sch"
-			(at 114.935 94.5646 0)
+			(at 120.65 116.1546 0)
 			(effects
 				(font
@@
 	)
 	(sheet
-		(at 43.815 74.93)
-		(size 19.685 20.32)
+		(at 120.65 69.85)
+		(size 27.94 20.32)
 		(exclude_from_sim no)
 		(in_bom yes)
@@
 		)
 		(property "Sheetname" "Motor and Hall"
-			(at 43.815 74.2184 0)
+			(at 120.65 69.1384 0)
 			(effects
 				(font
@@
 		)
 		(property "Sheetfile" "MotorHall.kicad_sch"
-			(at 43.815 95.8346 0)
+			(at 120.65 90.7546 0)
 			(effects
 				(font
@@
 	)
 	(sheet
-		(at 240.03 74.295)
-		(size 19.685 22.86)
+		(at 151.13 95.25)
+		(size 27.94 20.32)
 		(exclude_from_sim no)
 		(in_bom yes)
@@
 		)
 		(property "Sheetname" "Matrix"
-			(at 240.03 73.5834 0)
+			(at 151.13 94.5384 0)
 			(effects
 				(font
@@
 		)
 		(property "Sheetfile" "Matrix.kicad_sch"
-			(at 240.03 97.7396 0)
+			(at 151.13 116.1546 0)
 			(effects
 				(font
