File: PCB Rev 2/VolumetricDisplay.kicad_pcb (KiCad board)
At the start: 4 copper layers, 48.5 x 56 mm, 207 parts, among them J1 USB_C_Receptacle_USB2.0_16P, Q1 DMN32D2LDF, Q2 DMN32D2LDF, Q3 DMN32D2LDF, Q4 DMN32D2LDF, U1 FT260S-R, U2 NCP718xSN330, U3 STM32G071R8T6, U4 DRV8311S, U5 DRV5055A1xDBZxQ1

Commit message: started routing rev2
Parts:
- removed C6: 100nF, Capacitor_SMD:C_0402_1005Metric_Pad0.74x0.62mm_HandSolder
- removed R10, R11, R12, R13, R14, R15, R16, R17, R18, R19, R20, R21, R22, R23, R24, R25, R26, R27, R28, R29, R30, R31, R32, R33, R34, R35, R36, R37, R38, R39, R40, R41, R42, R43, R44, R45, R46, R47, R48, R49, R50, R51, R52, R53, R54, R55, R56, R57, R58, R59, R60, R61, R62, R63, R64, R9: 130, Resistor_SMD:R_0603_1608Metric_Pad0.98x0.95mm_HandSolder
- removed R100, R99: 100K, Resistor_SMD:R_0603_1608Metric_Pad0.98x0.95mm_HandSolder
- removed R68, R69, R70, R71, R72, R73: 0, Resistor_SMD:R_0402_1005Metric_Pad0.72x0.64mm_HandSolder
- removed R87, R88, R89, R90, R91, R92, R93, R94, R95: 0, Resistor_SMD:R_0603_1608Metric_Pad0.98x0.95mm_HandSolder
- removed TP1, TP2, TP3, TP4, TP5: TestPoint, TestPoint:TestPoint_Pad_D1.5mm
- removed U1: FT260S-R, Package_SO:TSSOP-28_4.4x9.7mm_P0.65mm
- added C11: 100nF, Capacitor_SMD:C_0402_1005Metric_Pad0.74x0.62mm_HandSolder, B.Cu at (137.3, 107.9)
- added C12: 100nF, Capacitor_SMD:C_0402_1005Metric_Pad0.74x0.62mm_HandSolder, B.Cu at (129.0, 100.3)
- added C13: 100nF, Capacitor_SMD:C_0402_1005Metric_Pad0.74x0.62mm_HandSolder, B.Cu at (137.7, 92.9)
- added C14: 100nF, Capacitor_SMD:C_0402_1005Metric_Pad0.74x0.62mm_HandSolder, B.Cu at (138.7, 92.9)
- added C15: 100nF, Capacitor_SMD:C_0402_1005Metric_Pad0.74x0.62mm_HandSolder, B.Cu at (129.7, 103.3)
- added C16: 100nF, Capacitor_SMD:C_0402_1005Metric_Pad0.74x0.62mm_HandSolder, B.Cu at (144.1, 102.5)
- added C17: 100nF, Capacitor_SMD:C_0402_1005Metric_Pad0.74x0.62mm_HandSolder, B.Cu at (129.4, 96.8)
- added C18: 100nF, Capacitor_SMD:C_0402_1005Metric_Pad0.74x0.62mm_HandSolder, B.Cu at (143.7, 98.2)
- added C19: 100nF, Capacitor_SMD:C_0402_1005Metric_Pad0.74x0.62mm_HandSolder, B.Cu at (144.2, 100.2)
- added C20: 100nF, Capacitor_SMD:C_0402_1005Metric_Pad0.74x0.62mm_HandSolder, B.Cu at (134.9, 107.5)
- added C21: 100nF, Capacitor_SMD:C_0402_1005Metric_Pad0.74x0.62mm_HandSolder, B.Cu at (129.2, 99.0)
- added C22: 4.7uF, Capacitor_SMD:C_0402_1005Metric_Pad0.74x0.62mm_HandSolder, B.Cu at (133.2, 92.5)
- added C23: 15pF, Capacitor_SMD:C_0402_1005Metric_Pad0.74x0.62mm_HandSolder, B.Cu at (131.0, 108.0)
- added C24: 15pF, Capacitor_SMD:C_0402_1005Metric_Pad0.74x0.62mm_HandSolder, B.Cu at (135.0, 109.5)
- added J2: Conn_ARM_SWD_TagConnect_TC2030, Connector:Tag-Connect_TC2030-IDC-NL_2x03_P1.27mm_Vertical, B.Cu at (125.2, 103.1)
- added L1: 3.3uH, Inductor_SMD:L_0805_2012Metric_Pad1.05x1.20mm_HandSolder, B.Cu at (133.4, 91.0)
- added R105: 33, Resistor_SMD:R_0603_1608Metric_Pad0.98x0.95mm_HandSolder, B.Cu at (130.3, 93.2)
- added Y1: Abracon ABM8-272-T3, Crystal:Crystal_SMD_Abracon_ABM8G-4Pin_3.2x2.5mm, B.Cu at (131.5, 110.5)
- C7: value 1uF -> 4.7uF; footprint Capacitor_SMD:C_0603_1608Metric_Pad1.08x0.95mm_HandSolder -> Capacitor_SMD:C_0402_1005Metric_Pad0.74x0.62mm_HandSolder
- J1, R66, R67: moved to F.Cu
- R1, R2, R3, R4, R5, R6, R7, R8: value 130 -> 50; moved to B.Cu
- U3: value STM32G071R8T6 -> RP2354B; footprint Package_QFP:LQFP-64_10x10mm_P0.5mm -> Package_DFN_QFN:QFN-80-1EP_10x10mm_P0.4mm_EP3.4x3.4mm
- moved R98 27.0 mm to (128.0, 77.0), turned to 90 degrees
- moved R84 25.5 mm to (154.7, 122.7), turned to 180 degrees
- moved R97 21.6 mm to (129.5, 77.0), turned to -90 degrees
- moved C5 20.9 mm to (133.2, 93.5), turned to 180 degrees
- moved C7 19.8 mm to (129.9, 95.4)
- moved R85 14.6 mm to (154.7, 121.2), turned to 180 degrees
- moved R66 14.0 mm to (129.1, 78.5), turned to 0 degrees
- moved R104 11.3 mm to (115.7, 126.8), turned to -90 degrees
- moved R86 10.7 mm to (153.8, 118.8), turned to -90 degrees
- moved U3 10.4 mm to (136.5, 100.4)
- moved J1 5.82 mm to (139.6, 81.0), turned to 180 degrees
- moved C4 4.73 mm to (139.5, 107.9), turned to -90 degrees
- moved R74 3.30 mm to (147.8, 114.2)
- moved R83 3.05 mm to (142.8, 117.2), turned to 0 degrees
- moved R77 3.02 mm to (150.0, 116.7), turned to 180 degrees
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Connections:
- net /Programming/VBUS renamed /MCU/VBUS
- C7 pad 1: GND -> Net-(U3-VREG_AVDD)
- C7 pad 2: Net-(U3-VREF+) -> GND
- D1 pad 1: FET0 -> Net-(D1-K)
- D1 pad 2: Net-(D1-A) -> LED0
- D10 pad 1: FET1 -> Net-(D10-K)
- D10 pad 2: Net-(D10-A) -> LED1
- D11 pad 1: FET2 -> Net-(D11-K)
- D11 pad 2: Net-(D11-A) -> LED1
- D12 pad 1: FET3 -> Net-(D12-K)
- D12 pad 2: Net-(D12-A) -> LED1
- D13 pad 1: FET4 -> Net-(D13-K)
- D13 pad 2: Net-(D13-A) -> LED1
- D14 pad 1: FET5 -> Net-(D14-K)
- D14 pad 2: Net-(D14-A) -> LED1
- D15 pad 1: FET6 -> Net-(D15-K)
- D15 pad 2: Net-(D15-A) -> LED1
- D16 pad 1: FET7 -> Net-(D16-K)
- D16 pad 2: Net-(D16-A) -> LED1
- D17 pad 1: FET0 -> Net-(D1-K)
- D17 pad 2: Net-(D17-A) -> LED2
- D18 pad 1: FET1 -> Net-(D10-K)
- D18 pad 2: Net-(D18-A) -> LED2
- D19 pad 1: FET2 -> Net-(D11-K)
- D19 pad 2: Net-(D19-A) -> LED2
- D2 pad 1: FET1 -> Net-(D10-K)
- D2 pad 2: Net-(D2-A) -> LED0
- D20 pad 1: FET3 -> Net-(D12-K)
- D20 pad 2: Net-(D20-A) -> LED2
- D21 pad 1: FET4 -> Net-(D13-K)
- D21 pad 2: Net-(D21-A) -> LED2
- D22 pad 1: FET5 -> Net-(D14-K)
- D22 pad 2: Net-(D22-A) -> LED2
- D23 pad 1: FET6 -> Net-(D15-K)
- D23 pad 2: Net-(D23-A) -> LED2
- D24 pad 1: FET7 -> Net-(D16-K)
- D24 pad 2: Net-(D24-A) -> LED2
- D25 pad 1: FET0 -> Net-(D1-K)
- D25 pad 2: Net-(D25-A) -> LED3
- D26 pad 1: FET1 -> Net-(D10-K)
- D26 pad 2: Net-(D26-A) -> LED3
- D27 pad 1: FET2 -> Net-(D11-K)
- D27 pad 2: Net-(D27-A) -> LED3
- D28 pad 1: FET3 -> Net-(D12-K)
- D28 pad 2: Net-(D28-A) -> LED3
- D29 pad 1: FET4 -> Net-(D13-K)
- D29 pad 2: Net-(D29-A) -> LED3
- D3 pad 1: FET2 -> Net-(D11-K)
- D3 pad 2: Net-(D3-A) -> LED0
- D30 pad 1: FET5 -> Net-(D14-K)
- D30 pad 2: Net-(D30-A) -> LED3
- D31 pad 1: FET6 -> Net-(D15-K)
- D31 pad 2: Net-(D31-A) -> LED3
- D32 pad 1: FET7 -> Net-(D16-K)
- D32 pad 2: Net-(D32-A) -> LED3
- D33 pad 1: FET0 -> Net-(D1-K)
- D33 pad 2: Net-(D33-A) -> LED4
- D34 pad 1: FET1 -> Net-(D10-K)
- D34 pad 2: Net-(D34-A) -> LED4
- D35 pad 1: FET2 -> Net-(D11-K)
- D35 pad 2: Net-(D35-A) -> LED4
- D36 pad 1: FET3 -> Net-(D12-K)
- D36 pad 2: Net-(D36-A) -> LED4
- D37 pad 1: FET4 -> Net-(D13-K)
- D37 pad 2: Net-(D37-A) -> LED4
- D38 pad 1: FET5 -> Net-(D14-K)
- D38 pad 2: Net-(D38-A) -> LED4
- D39 pad 1: FET6 -> Net-(D15-K)
- D39 pad 2: Net-(D39-A) -> LED4
- D4 pad 1: FET3 -> Net-(D12-K)
- D4 pad 2: Net-(D4-A) -> LED0
- D40 pad 1: FET7 -> Net-(D16-K)
- D40 pad 2: Net-(D40-A) -> LED4
- D41 pad 1: FET0 -> Net-(D1-K)
- D41 pad 2: Net-(D41-A) -> LED5
- D42 pad 1: FET1 -> Net-(D10-K)
- D42 pad 2: Net-(D42-A) -> LED5
- D43 pad 1: FET2 -> Net-(D11-K)
- D43 pad 2: Net-(D43-A) -> LED5
- D44 pad 1: FET3 -> Net-(D12-K)
- D44 pad 2: Net-(D44-A) -> LED5
- D45 pad 1: FET4 -> Net-(D13-K)
- D45 pad 2: Net-(D45-A) -> LED5
- D46 pad 1: FET5 -> Net-(D14-K)
- D46 pad 2: Net-(D46-A) -> LED5
- D47 pad 1: FET6 -> Net-(D15-K)
- D47 pad 2: Net-(D47-A) -> LED5
- D48 pad 1: FET7 -> Net-(D16-K)
- D48 pad 2: Net-(D48-A) -> LED5
- D49 pad 1: FET0 -> Net-(D1-K)
- D49 pad 2: Net-(D49-A) -> LED6
- D5 pad 1: FET4 -> Net-(D13-K)
- D5 pad 2: Net-(D5-A) -> LED0
- D50 pad 1: FET1 -> Net-(D10-K)
- D50 pad 2: Net-(D50-A) -> LED6
- D51 pad 1: FET2 -> Net-(D11-K)
- D51 pad 2: Net-(D51-A) -> LED6
- D52 pad 1: FET3 -> Net-(D12-K)
- D52 pad 2: Net-(D52-A) -> LED6
- D53 pad 1: FET4 -> Net-(D13-K)
- D53 pad 2: Net-(D53-A) -> LED6
- D54 pad 1: FET5 -> Net-(D14-K)
- D54 pad 2: Net-(D54-A) -> LED6
- D55 pad 1: FET6 -> Net-(D15-K)
- D55 pad 2: Net-(D55-A) -> LED6
- D56 pad 1: FET7 -> Net-(D16-K)
- D56 pad 2: Net-(D56-A) -> LED6
- D57 pad 1: FET0 -> Net-(D1-K)
- D57 pad 2: Net-(D57-A) -> LED7
- D58 pad 1: FET1 -> Net-(D10-K)
- D58 pad 2: Net-(D58-A) -> LED7
- D59 pad 1: FET2 -> Net-(D11-K)
- D59 pad 2: Net-(D59-A) -> LED7
- D6 pad 1: FET5 -> Net-(D14-K)
- D6 pad 2: Net-(D6-A) -> LED0
- D60 pad 1: FET3 -> Net-(D12-K)
- D60 pad 2: Net-(D60-A) -> LED7
- D61 pad 1: FET4 -> Net-(D13-K)
- D61 pad 2: Net-(D61-A) -> LED7
- D62 pad 1: FET5 -> Net-(D14-K)
- D62 pad 2: Net-(D62-A) -> LED7
- D63 pad 1: FET6 -> Net-(D15-K)
- D63 pad 2: Net-(D63-A) -> LED7
- D64 pad 1: FET7 -> Net-(D16-K)
- D64 pad 2: Net-(D64-A) -> LED7
- D7 pad 1: FET6 -> Net-(D15-K)
- D7 pad 2: Net-(D7-A) -> LED0
- D8 pad 1: FET7 -> Net-(D16-K)
- D8 pad 2: Net-(D8-A) -> LED0
- D9 pad 1: FET0 -> Net-(D1-K)
- D9 pad 2: Net-(D9-A) -> LED1
- R1 pad 1: Net-(D1-A) -> FET0
- R1 pad 2: LED0 -> Net-(D1-K)
- R2 pad 1: Net-(D2-A) -> FET1
- R2 pad 2: LED0 -> Net-(D10-K)
- R3 pad 1: Net-(D3-A) -> FET2
- R3 pad 2: LED0 -> Net-(D11-K)
- R4 pad 1: Net-(D4-A) -> FET3
- R4 pad 2: LED0 -> Net-(D12-K)
- R5 pad 1: Net-(D5-A) -> FET4
- R5 pad 2: LED0 -> Net-(D13-K)
- R6 pad 1: Net-(D6-A) -> FET5
- R6 pad 2: LED0 -> Net-(D14-K)
- R7 pad 1: Net-(D7-A) -> FET6
- R7 pad 2: LED0 -> Net-(D15-K)
- R74 pad 1: Net-(U3-PA1) -> Net-(U3-GPIO2)
- R75 pad 1: Net-(U3-PA2) -> Net-(U3-GPIO3)
- R76 pad 1: Net-(U3-PA3) -> Net-(U3-GPIO4)
- R77 pad 1: Net-(U3-PA4) -> Net-(U3-GPIO1)
- R78 pad 1: Net-(U3-PA5) -> Net-(U3-GPIO5)
- R79 pad 1: Net-(U3-PA6) -> Net-(U3-GPIO6)
- R8 pad 1: Net-(D8-A) -> FET7
- R8 pad 2: LED0 -> Net-(D16-K)
- R80 pad 1: Net-(U3-PA7) -> Net-(U3-GPIO7)
- R81 pad 1: Net-(U3-PA8) -> Net-(U3-GPIO8)
- R82 pad 1: Net-(U3-PA9/PA11) -> Net-(U3-GPIO9)
- R83 pad 1: Net-(U3-PA9/UCPD1_DBCC1) -> Net-(U3-GPIO10)
- R84 pad 1: Net-(U3-PA10/PA12) -> Net-(U3-GPIO11)
- R85 pad 1: Net-(U3-PA10/UCPD1_DBCC2) -> Net-(U3-GPIO12)
- R86 pad 1: Net-(U3-PD1) -> Net-(U3-GPIO0)
- R96 pad 1: Net-(U3-PA0) -> Net-(U3-GPIO41/ADC1)
- U3 pad 1: Net-(U3-PC11) -> Net-(U3-GPIO4)
- U3 pad 10: unconnected-(U3-PF0-Pad10) -> +1V1
- U3 pad 11: unconnected-(U3-PF1-Pad11) -> Net-(U3-GPIO12)
- U3 pad 12: nRST -> LED0
- U3 pad 13: Net-(U3-PC0) -> LED1
- U3 pad 14: Net-(U3-PC1) -> LED2
- U3 pad 15: Net-(U3-PC2) -> 3V3
- U3 pad 16: Net-(U3-PC3) -> LED3
- U3 pad 17: Net-(U3-PA0) -> LED4
- U3 pad 18: Net-(U3-PA1) -> LED5
- U3 pad 19: Net-(U3-PA2) -> LED6
- U3 pad 2: unconnected-(U3-PC12-Pad2) -> Net-(U3-GPIO5)
- U3 pad 20: Net-(U3-PA3) -> LED7
- U3 pad 21: Net-(U3-PA4) -> LED15
- U3 pad 22: Net-(U3-PA5) -> LED14
- U3 pad 23: Net-(U3-PA6) -> LED13
- U3 pad 24: Net-(U3-PA7) -> 3V3
- U3 pad 25: Net-(U3-PC4) -> LED12
- U3 pad 26: Net-(U3-PC5) -> LED11
- U3 pad 27: unconnected-(U3-PB0-Pad27) -> LED10
- U3 pad 28: unconnected-(U3-PB1-Pad28) -> LED9
- U3 pad 29: unconnected-(U3-PB2-Pad29) -> 3V3
- U3 pad 3: unconnected-(U3-PC13-Pad3) -> Net-(U3-GPIO6)
- U3 pad 30: unconnected-(U3-PB10-Pad30) -> Net-(U3-XIN)
- U3 pad 31: unconnected-(U3-PB11-Pad31) -> Net-(U3-XOUT)
- U3 pad 32: LED2 -> +1V1
- U3 pad 33: LED15 -> SWCLK
- U3 pad 34: LED14 -> SWDIO
- U3 pad 35: LED13 -> nRST
- U3 pad 36: Net-(U3-PA8) -> LED8
- U3 pad 37: Net-(U3-PA9/UCPD1_DBCC1) -> unconnected-(U3-GPIO29-Pad37)
- U3 pad 38: Net-(U3-PC6) -> unconnected-(U3-GPIO30-Pad38)
- U3 pad 39: LED12 -> unconnected-(U3-GPIO31-Pad39)
- U3 pad 4: unconnected-(U3-PC14-Pad4) -> Net-(U3-GPIO7)
- U3 pad 40: LED10 -> PRG_TX
- U3 pad 41: LED11 -> 3V3
- U3 pad 42: Net-(U3-PA10/UCPD1_DBCC2) -> PRG_RX
- U3 pad 43: Net-(U3-PA9/PA11) -> unconnected-(U3-GPIO34-Pad43)
- U3 pad 44: Net-(U3-PA10/PA12) -> unconnected-(U3-GPIO35-Pad44)
- U3 pad 45: SWDIO -> unconnected-(U3-GPIO36-Pad45)
- U3 pad 46: SWCLK -> unconnected-(U3-GPIO37-Pad46)
- U3 pad 47: LED0 -> unconnected-(U3-GPIO38-Pad47)
- U3 pad 48: LED1 -> unconnected-(U3-GPIO39-Pad48)
- U3 pad 5: unconnected-(U3-PC15-Pad5) -> 3V3
- U3 pad 50: LED8 -> 3V3
- U3 pad 51: Net-(U3-PD1) -> +1V1
- U3 pad 52: LED9 -> Net-(U3-GPIO41/ADC1)
- U3 pad 57: LED3 -> unconnected-(U3-GPIO46/ADC6-Pad57)
- U3 pad 59: unconnected-(U3-PB5-Pad59) -> 3V3
- U3 pad 6: unconnected-(U3-VBAT-Pad6) -> Net-(U3-GPIO8)
- U3 pad 60: LED4 -> 3V3
- U3 pad 61: LED5 -> Net-(U3-VREG_AVDD)
- U3 pad 62: LED7 -> GND
- U3 pad 63: LED6 -> Net-(U3-VREG_LX)
- U3 pad 64: Net-(U3-PC10) -> 3V3
- U3 pad 7: Net-(U3-VREF+) -> Net-(U3-GPIO9)
- U3 pad 8: 3V3 -> Net-(U3-GPIO10)
- U3 pad 9: GND -> Net-(U3-GPIO11)
Routing:
- net LED9: track 25.2 -> 131.7 mm
- net 3V3: track 129.3 -> 32.2 mm, vias 5 -> 17
- net FET7: track 67.1 -> 1.50 mm, vias 1 -> 0
- net FET2: track 60.7 -> 1.50 mm, vias 13 -> 0
- net FET1: track 57.6 -> 1.50 mm, vias 9 -> 0
- net FET5: track 55.5 -> 1.50 mm, vias 12 -> 0
- net Net-(D13-K): track 0.00 -> 53.5 mm, vias 0 -> 10
- net Net-(U3-PC0): track 53.0 -> 0.00 mm, vias 2 -> 0
- net FET6: track 54.0 -> 1.50 mm, vias 9 -> 0
- net FET4: track 53.5 -> 1.50 mm, vias 14 -> 0
- net Net-(D10-K): track 0.00 -> 51.7 mm, vias 0 -> 14
- net Net-(D12-K): track 0.00 -> 49.6 mm, vias 0 -> 9
- net FET3: track 50.8 -> 1.50 mm, vias 12 -> 0
- net Net-(D1-K): track 0.00 -> 47.5 mm, vias 0 -> 1
- net Net-(D11-K): track 0.00 -> 47.1 mm, vias 0 -> 14
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- added copper zone on F.Cu, net GND

Commit message: continued routing
Parts:
- moved C18 0.22 mm to (143.8, 98.0)
- moved C19 0.15 mm to (144.2, 100.4)
Routing:
- net Net-(U3-GPIO12): track 0.00 -> 63.6 mm, vias 0 -> 4
- net Net-(U3-GPIO0): track 0.00 -> 52.0 mm, vias 0 -> 4
- net LED9: track 131.7 -> 80.0 mm
- net Net-(U3-GPIO2): track 0.00 -> 51.1 mm, vias 0 -> 5
- net Net-(U3-GPIO5): track 0.00 -> 48.5 mm, vias 0 -> 6
- net Net-(D16-K): track 2.07 -> 50.5 mm
- net Net-(U3-GPIO11): track 0.00 -> 45.6 mm, vias 0 -> 2
- net Net-(U3-GPIO1): track 0.00 -> 44.3 mm, vias 0 -> 4
- net Net-(U3-GPIO3): track 0.00 -> 43.8 mm, vias 0 -> 4
- net Net-(U3-GPIO6): track 0.00 -> 42.5 mm, vias 0 -> 2
- net Net-(U3-GPIO7): track 0.00 -> 41.6 mm, vias 0 -> 2
- net Net-(U3-GPIO4): track 0.00 -> 37.9 mm, vias 0 -> 4
- net Net-(U3-GPIO9): track 0.00 -> 35.1 mm, vias 0 -> 4
- net Net-(U3-GPIO41/ADC1): track 0.00 -> 32.2 mm, vias 0 -> 4
- net Net-(U3-GPIO8): track 0.00 -> 30.5 mm, vias 0 -> 4
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
Commit message: more routing
Routing:
- net 5V: track 19.8 -> 24.8 mm, vias 6 -> 8
- net GND: vias 32 -> 34
Changed lines of the file:
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@@
+	)
+	(via
+		(at 157.65 97.75)
+		(size 0.6)
+		(drill 0.3)
+		(layers "F.Cu" "B.Cu")
+		(free yes)
+		(net "GND")
 	)
 	(via
@@
 	(via
 		(at 133.65 98.35)
+		(size 0.6)
+		(drill 0.3)
+		(layers "F.Cu" "B.Cu")
+		(free yes)
+		(net "GND")
+	)
+	(via
+		(at 159.75 98.55)
 		(size 0.6)
 		(drill 0.3)
@@
 	)
 	(via
+		(at 144.5875 86.3875)
+		(size 0.6)
+		(drill 0.3)
+		(layers "F.Cu" "B.Cu")
+		(net "5V")
+	)
+	(via
 		(at 148.5 82)
 		(size 0.6)
@@
 		)
 		(filling no)
+		(net "5V")
+	)
+	(via
+		(at 148.4 86.35)
+		(size 0.6)
+		(drill 0.3)
+		(layers "F.Cu" "B.Cu")
 		(net "5V")
 	)
@@
 	)
 	(segment
+		(start 147.775 86.35)
+		(end 147.4 86.725)
+		(width 0.75)
+		(layer "B.Cu")
+		(net "5V")
+	)
+	(segment
+		(start 148.4 86.35)
+		(end 147.775 86.35)
+		(width 0.75)
+		(layer "B.Cu")
+		(net "5V")
+	)
+	(segment
 		(start 150.201 127.19125)
 		(end 150.201 125.7315)
@@
 		(net "5V")
 	)
+	(segment
+		(start 144.5875 86.3875)
+		(end 148.3625 86.3875)
+		(width 0.75)
+		(layer "In2.Cu")
+		(net "5V")
+	)
+	(segment
+		(start 148.3625 86.3875)
+		(end 148.4 86.35)
+		(width 0.75)
+		(layer "In2.Cu")
+		(net "5V")
+	)

Commit message: Ryan Finished Routing
On my PC
Parts:
- added R68: 10K, Resistor_SMD:R_0603_1608Metric_Pad0.98x0.95mm_HandSolder, B.Cu at (126.7, 98.9)
- added R69: 10K, Resistor_SMD:R_0603_1608Metric_Pad0.98x0.95mm_HandSolder, B.Cu at (141.2, 85.8)
- added SW1: TS-1088-AR02016, TS-1088-AR02016:SW_TS-1088-AR02016, B.Cu at (123.8, 97.6)
- added SW2: TS-1088-AR02016, TS-1088-AR02016:SW_TS-1088-AR02016, B.Cu at (135.7, 84.8)
- moved G*** 0.40 mm to (152.9, 100.6)
- moved G*** 0.40 mm to (153.7, 95.6)
Routing:
- net Net-(D15-K): track 7.03 -> 65.4 mm, vias 2 -> 6
- net LED4: track 39.9 -> 77.7 mm, vias 2 -> 5
- net Net-(D14-K): track 20.7 -> 56.8 mm, vias 6 -> 10
- net 3V3: track 46.1 -> 78.8 mm, vias 18 -> 20
- net /MCU/QSPI_CS: track 0.00 -> 15.7 mm, vias 0 -> 2
- net 5V: track 24.8 -> 32.8 mm, vias 8 -> 10
- net nRST: track 11.6 -> 18.4 mm
- net GND: track 28.3 -> 33.3 mm, vias 34 -> 46
- net Net-(D10-K): track 51.7 -> 52.7 mm
- net Net-(D16-K): track 50.5 -> 51.1 mm
